File: cuves/hard/jard_c3/jard_c3.kicad_sch (KiCad schematic)
At the start: 24 parts, among them J1 Connecteur, J2 LEDs, Q1 BPC_IPP034N03L, U1 ESP32-C3_SUPERMINI_TH, U2 BPC_Alim3_3V, X1 Trou, X2 Trou

Commit message: Annotation erreurs
Other:
- note added: "Mettre un pont diviseur sur POW_MES Ajouter 2 capas en entrée de l'alim (1000 uF + 100nF)"
Changed lines of the file:
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@@
     (stroke (width 0) (type default))
+  )
+  (text "Mettre un pont diviseur sur POW_MES\nAjouter 2 capas en entrée de l'alim (1000 uF + 100nF)"
+    (at 168.91 137.16 0)
+    (effects (font (size 1.27 1.27)) (justify left bottom))
   )
   (global_label "LED_ROUGE" (shape output) (at 134.62 138.43 0)
