File: oyas/master_rs485/hard/bus.kicad_sch (KiCad schematic)
At the start: 28 parts, among them J3 POWER_OYAS_12V, J4 BUS_OYAS, J7 Adapt BUS, Q1 BPC_2N2222A, Q2 P03P4L-04, U4 BPC_Mod485

Commit message: Quelques commentaires sur le schéma pour préparer la version 2027...
Parts:
- R3: value 100 -> 220
Other:
- note added: "Ajouter grosse Capa 1000 µF sur 12V BUS Ajouter aussi une TVS 18V 600W sur 12V Bus"
- note added: "Pourquoi encore utiliser ces foutus modules ? => Remplacer par un CMS MAX485 5V"
Changed lines of the file:
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@@
     (effects (font (size 1.27 1.27) (thickness 0.254) bold) (justify left bottom))
+  )
+  (text "Ajouter grosse Capa 1000 µF sur 12V BUS\nAjouter aussi une TVS 18V 600W sur 12V Bus"
+    (at 231.14 148.59 0)
+    (effects (font (size 1.27 1.27)) (justify left bottom))
   )
   (text "R13 montée\nsi R7 du MOD485 non montée" (at 189.23 111.76 0)
@@
   )
   (text "A ajuster" (at 153.67 115.57 0)
+    (effects (font (size 1.27 1.27)) (justify left bottom))
+  )
+  (text "Pourquoi encore utiliser ces foutus modules ?\n=> Remplacer par un CMS MAX485 5V"
+    (at 53.975 90.805 0)
     (effects (font (size 1.27 1.27)) (justify left bottom))
   )
@@
       (effects (font (size 1.27 1.27)))
     )
-    (property "Value" "100" (at 152.4 51.6636 90)
+    (property "Value" "220" (at 152.4 51.6636 90)
       (effects (font (size 1.27 1.27)))
     )
