File: oyas/master_rs485/hard/cpu.kicad_sch (KiCad schematic)
At the start: 11 parts, among them J2 Log, J6 Button, U1 RtcArduino, U5 BPC_ESP8266-01_ESP-01

Commit message: Quelques commentaires sur le schéma pour préparer la version 2027...
Other:
- note added: "Ajouter capas de découplage pour le module ?"
- note added: "Attention, EN devrait être à 1. C'est miraculeux que ça marche !"
- note added: "Voir le découplage/filtrage 3.3V Adapter à l'ESP (Wifi = bursts)"
Changed lines of the file:
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@@
     (effects (font (size 5.08 5.08) (thickness 2.54) bold) (justify left bottom))
+  )
+  (text "Attention, EN devrait être à 1. C'est miraculeux que ça marche !"
+    (at 148.59 132.08 0)
+    (effects (font (size 1.27 1.27)) (justify left bottom))
+  )
+  (text "Voir le découplage/filtrage 3.3V\nAdapter à l'ESP (Wifi = bursts)"
+    (at 213.36 92.71 0)
+    (effects (font (size 1.27 1.27)) (justify left bottom))
+  )
+  (text "Ajouter capas de découplage pour le module ?" (at 95.25 20.32 0)
+    (effects (font (size 1.27 1.27)) (justify left bottom))
   )
   (global_label "TX_LOG" (shape input) (at 245.11 60.96 180) (fields_autoplaced)
