File: oyas/slaves_rs485/carte_m0/cao/jard_rs485_slave_m0.kicad_pcb (KiCad board)
At the start: 2 copper layers, 78.6 x 30 mm, 68 parts, among them J1 POWER, J2 Niveaux/Débit, J3 EV1, J5 BPC_PRG_FTSH-105-01-L-DV-K_1, Q1 BPC_FMMT38C, Q2 P03P4L-04, U1 BPC_Alim5V, U2 ATSAMD21G18A-A, U3 MAX3485, U4 AP1117-15

Commit message: Finalisation Future Rev B
Routing:
- net +3.3V: track 253.4 -> 258.3 mm
- net GND: vias 26 -> 30
Changed lines of the file:
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@@
   (title_block
     (title "Esclave OYA M0")
-    (date "2026-04-14")
+    (date "2026-05-13")
     (rev "B")
     (company "BPC")
@@
         (effects (font (size 1 1) (thickness 0.15)) (justify mirror))
     )
-    (fp_text value "BPC_PRG_FTSH-105-01-L-DV-K_1" (at 0.76 -5.475 90) (layer "B.Fab")
+    (fp_text value "BPC_PRG_FTSH-105-01-L-DV-K_1" (at 0.76 -5.475 90) (layer "B.Fab") hide
         (effects (font (size 1 1) (thickness 0.15)) (justify mirror))
     )
@@
   (via (at 152.72 111.26) (size 0.8) (drill 0.4) (layers "F.Cu" "B.Cu") (free) (net 1))
   (via (at 161.77 98.47) (size 0.8) (drill 0.4) (layers "F.Cu" "B.Cu") (free) (net 1))
+  (via (at 188.62 95.7) (size 0.8) (drill 0.4) (layers "F.Cu" "B.Cu") (free) (net 1))
+  (via (at 187 98.09) (size 0.8) (drill 0.4) (layers "F.Cu" "B.Cu") (free) (net 1))
   (via (at 142.66 92.42) (size 0.8) (drill 0.4) (layers "F.Cu" "B.Cu") (free) (net 1))
   (via (at 183.38 101.01) (size 0.8) (drill 0.4) (layers "F.Cu" "B.Cu") (free) (net 1))
@@
   (via (at 170.72 102.16) (size 0.8) (drill 0.4) (layers "F.Cu" "B.Cu") (net 1))
   (via (at 180.38 109.8) (size 0.8) (drill 0.4) (layers "F.Cu" "B.Cu") (free) (net 1))
+  (via (at 184.39 97.99) (size 0.8) (drill 0.4) (layers "F.Cu" "B.Cu") (free) (net 1))
   (via (at 144.86 96.53) (size 0.8) (drill 0.4) (layers "F.Cu" "B.Cu") (net 1))
   (via (at 149.58 99.82) (size 0.8) (drill 0.4) (layers "F.Cu" "B.Cu") (free) (net 1))
@@
   (via (at 164.85 106.4) (size 0.8) (drill 0.4) (layers "F.Cu" "B.Cu") (free) (net 1))
   (via (at 177.67 89.61) (size 0.8) (drill 0.4) (layers "F.Cu" "B.Cu") (free) (net 1))
+  (via (at 187.5 89.85) (size 0.8) (drill 0.4) (layers "F.Cu" "B.Cu") (free) (net 1))
   (segment (start 145.5625 95.8275) (end 144.86 96.53) (width 0.5) (layer "B.Cu") (net 1))
   (segment (start 146.69 95.8275) (end 145.5625 95.8275) (width 0.5) (layer "B.Cu") (net 1))
@@
   (segment (start 144.78 109.01) (end 144.79 109) (width 0.25) (layer "B.Cu") (net 17))
   (segment (start 142.09 109.01) (end 144.78 109.01) (width 0.25) (layer "B.Cu") (net 17))
+  (segment (start 190.98 95.86) (end 190.98 99.09) (width 0.5) (layer "F.Cu") (net 18))
   (segment (start 185.11 88.56) (end 188.87 88.56) (width 0.5) (layer "F.Cu") (net 18))
   (segment (start 181.782299 98.892299) (end 182.574598 98.1) (width 0.5) (layer "F.Cu") (net 18))
@@
   (segment (start 158.83 97.07) (end 157.17 97.07) (width 0.5) (layer "F.Cu") (net 18))
   (segment (start 190.98 108.38) (end 190.98 113.37) (width 0.25) (layer "F.Cu") (net 18))
+  (segment (start 188.73 98.19) (end 188.73 98.11) (width 0.25) (layer "F.Cu") (net 18))
   (segment (start 190.98 105.25) (end 190.98 106.25) (width 0.25) (layer "F.Cu") (net 18))
   (segment (start 181.782701 100.582701) (end 181.782299 100.582299) (width 0.5) (layer "F.Cu") (net 18))
@@
   (segment (start 182.48 88.56) (end 185.11 88.56) (width 0.5) (layer "F.Cu") (net 18))
   (segment (start 162.5 89.7) (end 164.52 87.68) (width 0.5) (layer "F.Cu") (net 18))
+  (segment (start 190.98 90.67) (end 190.98 95.86) (width 0.5) (layer "F.Cu") (net 18))
   (segment (start 147.19 99.55) (end 147.65 99.55) (width 0.5) (layer "F.Cu") (net 18))
+  (segment (start 188.73 98.11) (end 190.98 95.86) (width 0.25) (layer "F.Cu") (net 18))
   (segment (start 182.574598 98.1) (end 183.69 96.984598) (width 0.5) (layer "F.Cu") (net 18))
   (segment (start 189.68 105.83) (end 190.4 105.83) (width 0.25) (layer "F.Cu") (net 18))
@@
   (segment (start 188.17 107.27) (end 190.43 107.27) (width 0.5) (layer "F.Cu") (net 18))
   (segment (start 152.78 91.2) (end 152.78 97.9) (width 0.5) (layer "F.Cu") (net 18))
+  (segment (start 190.98 99.09) (end 190.98 106.72) (width 0.5) (layer "F.Cu") (net 18))
   (segment (start 164.52 87.68) (end 173.56 87.68) (width 0.5) (layer "F.Cu") (net 18))
   (segment (start 176.945 101.67) (end 179.004598 101.67) (width 0.25) (layer "F.Cu") (net 18))
@@
   (segment (start 190.98 109.12) (end 190.54 109.56) (width 0.25) (layer "F.Cu") (net 18))
   (segment (start 152.78 97.9) (end 152.68 98) (width 0.5) (layer "F.Cu") (net 18))
-  (segment (start 190.98 90.67) (end 190.98 106.72) (width 0.5) (layer "F.Cu") (net 18))
   (segment (start 189.61 113.74) (end 190.61 113.74) (width 0.25) (layer "F.Cu") (net 18))
   (segment (start 179.432701 102.932701) (end 181.782701 100.582701) (width 0.5) (layer "F.Cu") (net 18))
@@
   (segment (start 190.06 107.27) (end 188.17 107.27) (width 0.5) (layer "F.Cu") (net 18))
   (via (at 165.25 101.5) (size 0.8) (drill 0.4) (layers "F.Cu" "B.Cu") (net 18))
-  (via (at 185.11 88.56) (size 0.8) (drill 0.4) (layers "F.Cu" "B.Cu") (net 18))
   (via (at 170.5 95.75) (size 0.8) (drill 0.4) (layers "F.Cu" "B.Cu") (net 18))
   (via (at 147.19 99.55) (size 0.8) (drill 0.4) (layers "F.Cu" "B.Cu") (net 18))
@@
   (via (at 176.86 106.62) (size 0.8) (drill 0.4) (layers "F.Cu" "B.Cu") (net 18))
   (via (at 179.432701 102.932701) (size 0.8) (drill 0.4) (layers "F.Cu" "B.Cu") (net 18))
+  (via (at 188.73 98.19) (size 0.8) (drill 0.4) (layers "F.Cu" "B.Cu") (net 18))
   (via (at 155.77 97.86) (size 0.8) (drill 0.4) (layers "F.Cu" "B.Cu") (net 18))
   (via (at 167 100.5) (size 0.8) (drill 0.4) (layers "F.Cu" "B.Cu") (net 18))
@@
   (via (at 174.44 88.56) (size 0.8) (drill 0.4) (layers "F.Cu" "B.Cu") (net 18))
   (via (at 179.707299 100.967299) (size 0.8) (drill 0.4) (layers "F.Cu" "B.Cu") (net 18))
+  (segment (start 188.73 99.78) (end 188.73 98.19) (width 0.25) (layer "B.Cu") (net 18))
   (segment (start 155.77 97.86) (end 157.335 97.86) (width 0.25) (layer "B.Cu") (net 18))
   (segment (start 180.32 107.26) (end 177.5 107.26) (width 0.5) (layer "B.Cu") (net 18))
