File: oyas/slaves_rs485/carte_m0/cao/jard_rs485_slave_m0.kicad_sch (KiCad schematic)
At the start: 0 parts

Commit message: Finitions PCB
Other:
- title: Esclave Oya MSP430 -> Carte Oya M0
Changed lines of the file:
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@@
   (paper "A4")
   (title_block
-    (title "Esclave Oya MSP430")
-    (date "2025-05-08")
-    (rev "Rev B1")
+    (title "Carte Oya M0")
+    (date "2026-03-06")
+    (rev "Rev A")
     (company "BPC")
     (comment 1 "Alim 12V - Bus RS485 - cmd EV/Pompe - Niveaux - Débit")

Commit message: Fin de revue avec ajout d'une diode TVS 18V en entrée
Other:
- title: Carte Oya M0 -> Esclave Oya M0
Changed lines of the file:
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@@
   (paper "A4")
   (title_block
-    (title "Carte Oya M0")
-    (date "2026-03-06")
-    (rev "Rev A")
+    (title "Esclave Oya M0")
+    (date "2026-03-07")
+    (rev "A")
     (company "BPC")
-    (comment 1 "Alim 12V - Bus RS485 - cmd EV/Pompe - Niveaux - Débit")
-    (comment 2 "Mesure alim")
+    (comment 1 "Technologie avec M0 / Petite carte")
+    (comment 2 "Monitoring de tension d'alimentation")
+    (comment 3 "1 sortie 12V/5A - 2 entrées TOR (niveaux) ou 1 débimètre - 1 LED - RS485")
   )
   (text "ALIM\nE/S" (at 120.65 97.79 0)

Commit message: Finalisation Future Rev B
Other:
- title: Esclave Oya M0 -> Esclave Oya m0
Changed lines of the file:
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@@
   (paper "A4")
   (title_block
-    (title "Esclave Oya M0")
-    (date "2026-04-14")
+    (title "Esclave Oya m0")
+    (date "2026-05-13")
     (rev "B")
     (company "BPC")
@@
     (comment 3 "1 sortie 12V/5A - 2 entrées TOR (niveaux) ou 1 débimètre - 1 LED - RS485")
   )
+  (text_box "Rev B:\n- Inversion RX/TX\n- Chgt conn. prog."
+    (at 127 140.335 0) (size 26.035 8.255)
+    (stroke (width 0) (type default))
+    (fill (type none))
+    (effects (font (size 1.27 1.27)) (justify left top))
+  )
   (text "ALIM\nE/S" (at 120.65 97.79 0)
